File: kicad/chouchou_mx/chouchou_mx.kicad_pcb (KiCad board)
At the start: 2 copper layers, 204.9 x 113.7 mm, 51 parts

Commit message: update with thumb closer
Parts:
- moved S19 7.00 mm to (163.6, 181.8)
- moved S29 7.00 mm to (88.3, 181.8)
- moved S39 7.00 mm to (163.6, 181.8)
- moved S9 7.00 mm to (88.3, 181.8)
- moved _7 7.00 mm to (92.1, 197.1)
- moved _8 7.00 mm to (159.8, 197.1)
- moved S10 7.00 mm to (105.8, 189.3)
- moved S20 7.00 mm to (146.1, 189.3)
- moved S30 7.00 mm to (105.8, 189.3)
- moved S40 7.00 mm to (146.1, 189.3)
- moved G*** 1.80 mm to (111.0, 164.0)
- moved G*** 0.90 mm to (141.0, 165.0)
Routing:
- net GP7: track 89.9 -> 103.1 mm, vias 1 -> 0
- net GND: track 588.0 -> 575.3 mm, vias 0 -> 1
- net GP11: track 79.1 -> 71.0 mm
- net GP9: track 40.6 -> 33.0 mm
- net GP26: track 101.7 -> 107.8 mm
- net GP8: track 56.1 -> 52.2 mm
- net GP1: track 48.8 -> 46.4 mm
- net GP10: track 64.4 -> 63.2 mm
- net GP28: track 61.9 -> 63.0 mm
Other:
- board size 204.9 x 113.7 mm -> 204.9 x 107.4 mm

Commit message: addition of mx pdf
Parts:
- moved S11 86.3 mm to (301.6, 134.9)
- moved S31 86.3 mm to (301.6, 134.9)
- moved G*** 86.3 mm to (197.3, 162.3)
- moved G*** 86.3 mm to (227.3, 163.3)
- moved S1 86.3 mm to (122.9, 134.9)
- moved S13 86.3 mm to (279.0, 130.3)
- moved S17 86.3 mm to (244.4, 148.3)
- moved S18 86.3 mm to (236.0, 131.2)
- moved S19 86.3 mm to (249.9, 180.1)
- moved S2 86.3 mm to (129.4, 117.0)
- moved S21 86.3 mm to (122.9, 134.9)
- moved S22 86.3 mm to (129.4, 117.0)
- moved S25 86.3 mm to (165.5, 133.0)
- moved S26 86.3 mm to (173.2, 115.6)
- moved S33 86.3 mm to (279.0, 130.3)
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
Commit message: update on the gerber for minimx and start of code for the french chouchou using kmk
Routing:
- net GP12: track 103.4 -> 113.6 mm
- net GND: track 575.3 -> 582.1 mm
Changed lines of the file:
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@@
 		(tenting front back)
 		(pcbplotparams
-			(layerselection 0x00000000_00000000_5555555f_ffffffff)
+			(layerselection 0x00000000_00000000_5555555f_5755f5ff)
 			(plot_on_all_layers_selection 0x00000000_00000000_00000000_00000000)
 			(disableapertmacros no)
-			(usegerberextensions no)
-			(usegerberattributes yes)
-			(usegerberadvancedattributes yes)
-			(creategerberjobfile yes)
+			(usegerberextensions yes)
+			(usegerberattributes no)
+			(usegerberadvancedattributes no)
+			(creategerberjobfile no)
 			(dashed_line_dash_ratio 12.000000)
 			(dashed_line_gap_ratio 3.000000)
@@
 			(sketchdnponfab yes)
 			(crossoutdnponfab yes)
-			(subtractmaskfromsilk no)
+			(subtractmaskfromsilk yes)
 			(outputformat 1)
 			(mirror no)
@@
 	)
 	(segment
+		(start 116.117652 136.154842)
+		(end 118.757617 138.794807)
+		(width 0.25)
+		(layer "B.Cu")
+		(net 1)
+	)
+	(segment
+		(start 117.092909 130.079868)
+		(end 116.117652 131.055125)
+		(width 0.25)
+		(layer "B.Cu")
+		(net 1)
+	)
+	(segment
+		(start 116.117652 131.055125)
+		(end 116.117652 136.154842)
+		(width 0.25)
+		(layer "B.Cu")
+		(net 1)
+	)
+	(segment
 		(start 243.5479 190.1428)
 		(end 233.4557 190.1428)
@@
 	)
 	(segment
+		(start 305.310322 132.189678)
+		(end 305.15185 132.34815)
+		(width 0.25)
+		(layer "B.Cu")
+		(net 2)
+	)
+	(segment
 		(start 179.4726 142.6727)
 		(end 179.4726 119.489)
@@
 	)
 	(segment
+		(start 305.15185 132.34815)
+		(end 302.65185 132.34815)
+		(width 0.25)
+		(layer "B.Cu")
+		(net 2)
+	)
+	(segment
 		(start 125.5934 138.5798)
 		(end 125.5934 136.6299)
@@
 	)
 	(segment
+		(start 302.65185 132.34815)
+		(end 302.0347 131.731)
+		(width 0.25)
+		(layer "B.Cu")
+		(net 2)
+	)
+	(segment
 		(start 275.3662 105.773)
 		(end 276.1993 107.835)
@@
 	)
 	(segment
+		(start 305.310322 128.11818)
+		(end 305.310322 132.189678)
+		(width 0.25)
+		(layer "B.Cu")
+		(net 2)
+	)
+	(segment
 		(start 247.4073 141.1552)
 		(end 246.4743 139.2424)
@@
 	(segment
 		(start 306.0071 135.7034)
-		(end 302.0347 131.731)
+		(end 302.65185 132.34815)
 		(width 0.25)
 		(layer "B.Cu")
